File: simple-p4.kicad_sch (KiCad schematic)
At the start: 0 parts

Commit message: Implement schematic for basic ESP32-P4 nets
Parts:
- added C11, C14, C20, C28: 10uF, symbol Device:C
- added C12, C13, C15, C16, C21, C23, C24, C26, C29, C31, C38, C6, C7, C8, C9: 0.1uF, symbol Device:C
- added C17, C18, C19, C22: 1uF, 1uF, symbol Device:C
- added C27, C30: 1uF, symbol Device:C
- added C32: 10nF, 1uF, symbol Device:C
- added C33: 0.1uF, 1uF, symbol Device:C
- added C34: 4.7uF, 1uF, symbol Device:C
- added R28: 10k, symbol Device:R
- added TP1: VDDO_FLASH, symbol Connector:TestPoint
- added TP2: VDDO4, symbol Connector:TestPoint
- added TP3: VDDO_PSRAM, symbol Connector:TestPoint
- added TP4: VDDO3, symbol Connector:TestPoint
- added U1: ~, PCM_Espressif:Espressif:ESP32-P4, symbol Espressif:ESP32-P4
- added U2: W25Q128JVS, Package_SO:SOIC-8_5.3x5.3mm_P1.27mm, symbol Memory_Flash:W25Q128JVS
- added U3: TLV62569DBV, Package_TO_SOT_SMD:SOT-23-5, symbol Regulator_Switching:TLV62569DBV
Connections:
- new net +3V3: C13.1, C14.1, C16.1, C20.1, C21.1, C23.1, C24.2, C32.1, C33.1, C34.1, C6.1, C7.1, C9.1, U1.101 (VDDA), U1.21 (VDDPST_2), U1.51 (VCCA), U1.62 (VDDPST_4), U1.75 (VDDPST_LDO), U1.77 (VDDPST_DCDC), U1.85 (VDDPST_5), U1.9 (VDDPST_1), U1.96 (VDDPST_6)
- new net CHIP_PU: U1.103 (CHIP_PU)
- new net EN_DCDC: U1.79 (EN_DCDC)
- new net ESP_VBAT: C11.1, C12.1, U1.102 (VBAT)
- new net ESP_VDD_HP: C15.1, C28.1, C29.1, C8.1, U1.26 (VDD_HP_0), U1.76 (VDD_HP_2), U1.91 (VDD_HP_3)
- new net FB_DCDC: U1.78 (FB_DCDC)
- new net FLASH_CK: U1.32 (FLASH_CK), U2.6 (CLK)
- new net FLASH_CS: R28.1, U1.27 (FLASH_CS), U2.1 (~{CS})
- new net FLASH_D: U1.33 (FLASH_D), U2.5 (DI/IO_{0})
- new net FLASH_HD: U1.31 (FLASH_HOLD), U2.7 (~{HOLD}/~{RESET}/IO_{3})
- new net FLASH_Q: U1.28 (FLASH_Q), U2.2 (DO/IO_{1})
- new net FLASH_WP: U1.29 (FLASH_WP), U2.3 (~{WP}/IO_{2})
- new net GND: C11.2, C12.2, C13.2, C14.2, C15.2, C16.2, C17.2, C18.2, C19.2, C20.2, C21.2, C22.2, C23.2, C24.1, C26.2, C27.2, C28.2, C29.2, C30.2, C31.2, C32.2, C33.2, C34.2, C38.2, C6.2, C7.2, C8.2, C9.2, U2.4 (GND)
- new net GPIO0: U1.104 (GPIO0/ADC)
- new net GPIO1: U1.1 (GPIO1/ADC)
- new net GPIO10: U1.11 (GPIO10/ADC)
- new net GPIO11: U1.12 (GPIO11/ADC)
- new net GPIO12: U1.13 (GPIO12/ADC)
- new net GPIO13: U1.14 (GPIO13/ADC)
- new net GPIO14: U1.15 (GPIO14/ADC)
- new net GPIO15: U1.16 (GPIO15/ADC)
- new net GPIO16: U1.17 (GPIO16/ADC)
- new net GPIO17: U1.18 (GPIO17/ADC)
- new net GPIO18: U1.19 (GPIO18/ADC)
- new net GPIO19: U1.20 (GPIO19/ADC)
- new net GPIO2: U1.2 (GPIO2/ADC)
- new net GPIO20: U1.22 (GPIO20/ADC)
- new net GPIO21: U1.23 (GPIO21/ADC)
- new net GPIO22: U1.24 (GPIO22/ADC)
- new net GPIO23: U1.25 (GPIO23/ADC)
- new net GPIO24: U1.52 (GPIO24/ADC/USB)
- new net GPIO25: U1.53 (GPIO25/ADC/USB)
- new net GPIO26: U1.55 (GPIO26/ADC/USB)
- new net GPIO27: U1.56 (GPIO27/ADC/USB)
- new net GPIO28: U1.57 (GPIO28)
- new net GPIO29: U1.58 (GPIO29)
- new net GPIO3: U1.3 (GPIO3/ADC)
- new net GPIO30: U1.60 (GPIO30)
- new net GPIO31: U1.61 (GPIO31)
- new net GPIO32: U1.63 (GPIO32)
- new net GPIO33: U1.64 (GPIO33)
- new net GPIO34: U1.65 (GPIO34)
- new net GPIO35: U1.66 (GPIO35)
- new net GPIO36: U1.68 (GPIO36)
- new net GPIO37: U1.69 (GPIO37)
- new net GPIO38: U1.70 (GPIO38)
- new net GPIO39: U1.80 (GPIO39)
- new net GPIO4: U1.4 (GPIO4/ADC)
- new net GPIO40: U1.81 (GPIO40)
- new net GPIO41: U1.82 (GPIO41)
- new net GPIO43: U1.84 (GPIO43)
- new net GPIO44: U1.86 (GPIO44)
- new net GPIO45: U1.87 (GPIO45)
- new net GPIO46: U1.88 (GPIO46)
- new net GPIO47: U1.89 (GPIO47)
- new net GPIO48: U1.90 (GPIO48)
- new net GPIO49: U1.92 (GPIO49/ADC)
- new net GPIO5: U1.5 (GPIO5/ADC)
- new net GPIO50: U1.93 (GPIO50/ADC)
- new net GPIO51: U1.94 (GPIO51/ADC)
- new net GPIO52: U1.83 (GPIO42), U1.95 (GPIO52/ADC)
- new net GPIO53: U1.97 (GPIO53/ADC)
- new net GPIO54: U1.98 (GPIO54/ADC)
- new net GPIO6: U1.6 (GPIO6/ADC)
- new net GPIO7: U1.7 (GPIO7/ADC)
- new net GPIO8: U1.8 (GPIO8/ADC)
- new net GPIO9: U1.10 (GPIO9/ADC)
- new net USB_DM: U1.49 (USB-DM)
- new net USB_DP: U1.50 (USB-DP)
- new net VDDO3: C19.1, TP4.1, U1.73 (VFB/VO3)
- new net VDDO4: C22.1, TP2.1, U1.74 (VFB/VO4)
- new net VDDO_FLASH: C17.1, C30.1, C31.1, TP1.1, U1.30 (VDDPST_3), U1.71 (VFB/VO1)
- new net VDDO_PSRAM: C18.1, C26.1, C27.1, TP3.1, U1.59 (VDDPST), U1.67 (VDDPST), U1.72 (VFB/VO2)
- new net VDD_FLASH: C38.1, R28.2, U2.8 (VCC)
- new net XTAL_N: U1.99 (XTAL_N)
- new net XTAL_P: U1.100 (XTAL_P)
Other:
- note added: "* Espressif said ETA3485, SY8088 and RY3420 should also work, footprint looks the same (SOT23-5) * Waveshare also tested MP1605GTF-Z, Iq is only 11uA??? (lowest of all) but Espressif didn't say it work * ETA3485 and TLV62569 looks good to me"
- note added: "* VDD_IO0"
- note added: "* VDD_LP"

Commit message: schematic: add crystal
Parts:
- added C1, C3: 10uF, symbol Device:C
- added C10, C25: 20pF, symbol Device:C
- added C2: NC, symbol Device:C
- added C35, C36: 0.1uF, symbol Device:C
- added C4, C5: 22pF, symbol Device:C
- added J1: Conn_01x26_Pin, symbol Connector:Conn_01x26_Pin
- added J2, J3: Conn_01x20_Pin, symbol Connector:Conn_01x20_Pin
- added J4: UART_PROG, Connector_PinHeader_2.54mm:PinHeader_1x06_P2.54mm_Vertical, symbol Connector:Conn_01x06_Pin
- added L1: 2.2uH/3A, symbol Device:L
- added R1, R2: NC, symbol Device:R
- added R3, R4: 10k, symbol Device:R
- added SW1: BOOT, symbol Switch:SW_Push
- added SW2: RST, symbol Switch:SW_Push
- added Y1: 40MHz 10ppm, symbol Device:Crystal_GND24
- added Y2: 32.768k, symbol Device:Crystal
Connections:
- net +3V3: now also U3.4 (VIN), C1.1, J1.26 (Pin_26), J2.19 (Pin_19), J2.20 (Pin_20), J3.20 (Pin_20), J4.1 (Pin_1), R3.1, R4.1
- net CHIP_PU: now also C36.1, J4.4 (Pin_4), R4.2, SW2.2
- net EN_DCDC: now also U3.1 (EN)
- net ESP_VDD_HP: now also C2.1, C3.1, L1.2, R1.1
- net FB_DCDC: now also U3.5 (FB), C2.2, R1.2, R2.1
- net GND: now also U3.2 (GND), C1.2, C10.1, C25.2, C3.2, C35.2, C36.2, C4.1, C5.2, J1.1 (Pin_1), J1.21 (Pin_21), J1.9 (Pin_9), J2.10 (Pin_10), J2.15 (Pin_15), J2.2 (Pin_2), J2.7 (Pin_7), J3.14 (Pin_14), J3.3 (Pin_3), J3.8 (Pin_8), J4.6 (Pin_6), R2.2, SW1.1, SW2.1, Y1.2, Y1.4
- net GPIO0: now also C10.2, Y2.1
- net GPIO1: now also C25.1, Y2.2
- net GPIO10: now also J1.11 (Pin_11)
- net GPIO11: now also J1.12 (Pin_12)
- net GPIO12: now also J1.13 (Pin_13)
- net GPIO13: now also J1.14 (Pin_14)
- net GPIO14: now also J1.15 (Pin_15)
- net GPIO15: now also J1.16 (Pin_16)
- net GPIO16: now also J1.17 (Pin_17)
- net GPIO17: now also J1.18 (Pin_18)
- net GPIO18: now also J1.19 (Pin_19)
- net GPIO19: now also J1.20 (Pin_20)
- net GPIO2: now also J1.2 (Pin_2)
- net GPIO20: now also J1.22 (Pin_22)
- net GPIO21: now also J1.23 (Pin_23)
- net GPIO22: now also J1.24 (Pin_24)
- net GPIO23: now also J1.25 (Pin_25)
- net GPIO25: now also J2.1 (Pin_1)
- net GPIO26: now also J2.3 (Pin_3)
- net GPIO27: now also J2.4 (Pin_4)
- net GPIO28: now also J2.5 (Pin_5)
- net GPIO29: now also J2.6 (Pin_6)
- net GPIO3: now also J1.3 (Pin_3)
- net GPIO30: now also J2.8 (Pin_8)
- net GPIO31: now also J2.9 (Pin_9)
- net GPIO32: now also J2.11 (Pin_11)
- net GPIO33: now also J2.12 (Pin_12)
- net GPIO34: now also J2.13 (Pin_13)
- net GPIO36: now also J2.16 (Pin_16)
- net GPIO39: now also J3.19 (Pin_19)
- net GPIO4: now also J1.4 (Pin_4)
- net GPIO40: now also J3.18 (Pin_18)
- net GPIO41: now also J3.17 (Pin_17)
- net GPIO43: now also J3.15 (Pin_15)
- net GPIO44: now also J3.13 (Pin_13)
- net GPIO45: now also J3.12 (Pin_12)
- net GPIO46: now also J3.11 (Pin_11)
- net GPIO47: now also J3.10 (Pin_10)
- net GPIO48: now also J3.9 (Pin_9)
- net GPIO49: now also J3.7 (Pin_7)
- net GPIO5: now also J1.5 (Pin_5)
- net GPIO50: now also J3.6 (Pin_6)
- net GPIO51: now also J3.5 (Pin_5)
- net GPIO52: now also J3.16 (Pin_16), J3.4 (Pin_4)
- net GPIO53: now also J3.2 (Pin_2)
- net GPIO54: now also J3.1 (Pin_1)
- net GPIO6: now also J1.6 (Pin_6)
- net GPIO7: now also J1.7 (Pin_7)
- net GPIO8: now also J1.8 (Pin_8)
- net GPIO9: now also J1.10 (Pin_10)
- net XTAL_N: now also C5.1, Y1.3
- net XTAL_P: now also C4.2, Y1.1
- net at U3.3 (SW): now also L1.1
- net GPIO35 renamed GPIO35/BOOT
- net GPIO35/BOOT: now also C35.1, J2.14 (Pin_14), J4.5 (Pin_5), R3.2, SW1.2
- net GPIO37 renamed GPIO37/U0TXD
- net GPIO37/U0TXD: now also J2.17 (Pin_17), J4.2 (Pin_2)
- net GPIO38 renamed GPIO38/U0RXD
- net GPIO38/U0RXD: now also J2.18 (Pin_18), J4.3 (Pin_3)
Other:
- note added: "* CL=12.5pF"
- note added: "* CL=15pF"
- note added: "* GPIO35 is BOOT pin"
- moved on the sheet: C11, C12, C13, C14, C15, C16, C17, C18, C19, C20, C21, C22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

Commit message: schematic: add USB port
Parts:
- added C37, C41: 10uF, Capacitor_SMD:C_0603_1608Metric, symbol Device:C_Small
- added C39, C40: 0.1uF, Capacitor_SMD:C_0402_1005Metric, symbol Device:C_Small
- added J5: USB_HS, Connector_USB:USB_C_Receptacle_HRO_TYPE-C-31-M-12, symbol Connector:USB_C_Receptacle_USB2.0
- added J6: USB_JTAG, Connector_USB:USB_C_Receptacle_HRO_TYPE-C-31-M-12, symbol Connector:USB_C_Receptacle_USB2.0
- added JP1: 3V3PWR, Jumper:SolderJumper-2_P1.3mm_Bridged_Pad1.0x1.5mm, symbol Jumper:Jumper_2_Bridged
- added R10, R5, R6, R9: 5.11k, Resistor_SMD:R_0402_1005Metric, symbol Device:R_Small
- added R7, R8: 0R, Resistor_SMD:R_0402_1005Metric, symbol Device:R_Small
- added U4: AP7361C-33E, Package_TO_SOT_SMD:SOT-223-3_TabPin2, symbol Regulator_Linear:AP7361C-33E
- C1, C11, C14, C20, C27, C28, C3, C30: footprint (none) -> Capacitor_SMD:C_0603_1608Metric
- C10, C12, C13, C15, C16, C2, C21, C23, C24, C25, C26, C29, C31, C35, C36, C38, C4, C5, C6, C7, C8, C9: footprint (none) -> Capacitor_SMD:C_0402_1005Metric
- C17, C18, C19, C22, C34: footprint 1uF -> Capacitor_SMD:C_0603_1608Metric
- C32, C33: footprint 1uF -> Capacitor_SMD:C_0402_1005Metric
- R1, R2, R3, R4: footprint (none) -> Resistor_SMD:R_0402_1005Metric
- R11: renamed from R28; footprint (none) -> Resistor_SMD:R_0402_1005Metric
- U1: footprint PCM_Espressif:Espressif:ESP32-P4 -> PCM_Espressif:Espressif_ESP32-P4
Connections:
- net +3V3: now also JP1.2 (B)
- net GND: now also U1.105 (GND), C37.2, C39.2, C40.2, C41.2, J5.A1 (GND), J5.A12 (GND), J5.B1 (GND), J5.B12 (GND), J5.S1 (SHIELD), J6.A1 (GND), J6.A12 (GND), J6.B1 (GND), J6.B12 (GND), J6.S1 (SHIELD), R10.2, R5.2, R6.2, R9.2, U4.2 (GND)
- net GPIO24: now also J6.A7 (D-), J6.B7 (D-)
- net GPIO25: now also J6.A6 (D+), J6.B6 (D+)
- net USB_DM: now also R7.1
- net USB_DP: now also R8.2
- new net: J5.B5 (CC2), R5.1
- new net: C40.1, C41.1, JP1.1 (A), U4.3 (VO)
- new net: J5.A6 (D+), J5.B6 (D+), R8.1
- new net: J5.A5 (CC1), R6.1
- new net: J5.A7 (D-), J5.B7 (D-), R7.2
- new net: J6.A5 (CC1), R10.1
- new net: J6.B5 (CC2), R9.1
- new net +5V: C37.1, C39.1, J5.A4 (VBUS), J5.A9 (VBUS), J5.B4 (VBUS), J5.B9 (VBUS), J6.A4 (VBUS), J6.A9 (VBUS), J6.B4 (VBUS), J6.B9 (VBUS), U4.1 (VI)
- no-connect marks 0 -> 4
Other:
- note added: "5v to 3.3v LDO"
- moved on the sheet: C1, C10, C2, C25, C3, C32, C33, C34, C35, C36, C38, C4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

Commit message: Finish PCB
Parts:
- removed C2: NC, Capacitor_SMD:C_0402_1005Metric, symbol Device:C
- removed J2, J3: Conn_01x20_Pin, symbol Connector:Conn_01x20_Pin
- removed R2: NC, Resistor_SMD:R_0402_1005Metric, symbol Device:R
- removed TP1: VDDO_FLASH, symbol Connector:TestPoint
- removed TP2: VDDO4, symbol Connector:TestPoint
- removed TP3: VDDO_PSRAM, symbol Connector:TestPoint
- removed TP4: VDDO3, symbol Connector:TestPoint
- added C42: 0.1uF, Capacitor_SMD:C_0402_1005Metric, symbol Device:C
- added J3: Micro_SD_Card_Det_Hirose_DM3AT, Connector_Card:microSD_HC_Hirose_DM3AT-SF-PEJM5, symbol Connector:Micro_SD_Card_Det_Hirose_DM3AT
- added JP2: VBAT, Jumper:SolderJumper-2_P1.3mm_Bridged_Pad1.0x1.5mm, symbol Jumper:Jumper_2_Bridged
- added R12, R13, R14, R15, R16, R17, R18, R19: 10k, Resistor_SMD:R_0402_1005Metric, symbol Device:R
- C1, C3: value 10uF -> 22uF
- J1: footprint (none) -> Connector_PinHeader_2.54mm:PinHeader_2x13_P2.54mm_Vertical
- L1: footprint (none) -> Inductor_SMD:L_Changjiang_FTC322510S
- R1: value NC -> 10k; now fitted
- SW1, SW2: footprint (none) -> Button_Switch_SMD:SW_Push_1P1T_XKB_TS-1187A
- U1: value ~ -> ESP32-P4; footprint PCM_Espressif:Espressif_ESP32-P4 -> Espressif:ESP32-P4
- Y1: footprint (none) -> Crystal:Crystal_SMD_2016-4Pin_2.0x1.6mm
- Y2: footprint (none) -> Crystal:Crystal_SMD_3215-2Pin_3.2x1.5mm
- renumbered J4 to J2, R4 to R2
Connections:
- net VDD_FLASH is gone; now on net VDDO_FLASH: C38.1, R11.2, U2.8 (VCC)
- net +3V3: now also R1.1, J3.4 (VDD), JP2.1 (A), R12.1, R13.1, R14.1, R15.1, R16.1, R17.1, R18.1, R19.1
- net CHIP_PU: now also C42.1, R12.2
- net FB_DCDC: no longer R1.2
- net GND: now also C42.2, J3.10 (DET_A), J3.11 (SHIELD), J3.6 (VSS)
- net GPIO39: now also J3.7 (DAT0), R17.2
- net GPIO40: now also J3.8 (DAT1), R18.2
- net GPIO41: now also J3.1 (DAT2), R13.2
- net GPIO43: now also J3.5 (CLK), R16.2
- net GPIO44: now also J3.3 (CMD), R15.2
- net GPIO45: now also J3.9 (DET_B), R19.2
- net GPIO52: no longer U1.83 (GPIO42)
- net ESP_VBAT: no longer names the net of C11.1, C12.1, U1.102 (VBAT)
- net ESP_VBAT: now also JP2.2 (B)
- net ESP_VDD_HP renamed +1V2
- net +1V2: no longer R1.1
- net GPIO26: no longer names the net of U1.55 (GPIO26/ADC/USB)
- net GPIO27: no longer names the net of U1.56 (GPIO27/ADC/USB)
- net GPIO28: no longer names the net of U1.57 (GPIO28)
- net GPIO29: no longer names the net of U1.58 (GPIO29)
- net GPIO30: no longer names the net of U1.60 (GPIO30)
- net GPIO31: no longer names the net of U1.61 (GPIO31)
- net GPIO32: no longer names the net of U1.63 (GPIO32)
- net GPIO33: no longer names the net of U1.64 (GPIO33)
- net GPIO34: no longer names the net of U1.65 (GPIO34)
- net GPIO36: no longer names the net of U1.68 (GPIO36)
- net GPIO36: now also R1.2
- new net GPIO42: J3.2 (DAT3/CD), R14.2, U1.83 (GPIO42)
- no-connect marks 4 -> 28
Other:
- note added: "Simple ESP32-P4 Dev board By Jackson Ming Hu <huming2207@gmail.com> Copright (C) 2025"
- moved on the sheet: C10, C24, C25, C28, C29, C3, C35, C36, C38, C4, C5, J2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
