File: simple-p4.kicad_pcb (KiCad board)
At the start: 4 copper layers, 50 x 65.5 mm, 75 parts, among them J1 Conn_01x26_Pin, J2 UART_PROG, J3 Micro_SD_Card_Det_Hirose_DM3AT, J5 USB_HS, J6 USB_JTAG, SW1 BOOT, SW2 RST, U1 ESP32-P4, U2 W25Q128JVS, U3 TLV62569DBV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

Commit message: Finish off PCB
Parts:
- moved C27 1.67 mm to (160.6, 107.8)
- moved C26 1.08 mm to (159.6, 105.7)
- moved R1 0.34 mm to (162.8, 105.3)
Connections:
- R1 pad 1: +3.3V -> +3V3
Routing:
- net GND: track 87.2 -> 113.7 mm, vias 36 -> 412
- net +3V3: track 50.2 -> 57.6 mm, vias 14 -> 20
- net +5V: track 40.0 -> 42.1 mm
- net GPIO0: track 4.90 -> 6.45 mm
- net FLASH_HD: track 7.44 -> 8.69 mm
- net +3.3V: track 1.01 -> 0.00 mm, vias 1 -> 0
- net CHIP_PU: track 65.5 -> 66.4 mm
- net VDDO_PSRAM: track 27.5 -> 26.7 mm
- net Net-(J5-CC2): track 6.43 -> 7.03 mm
- net GPIO25: track 23.5 -> 23.0 mm
Other:
- board size 50 x 65.5 mm -> 50 x 65.1 mm
- board text added: "NOT FOR RESELL UNLESS AUTHORISED BY THE AUTHOR"
- board text added: "SimpleP4 By Jackson M Hu Rev. 1, Sep 2025"

Commit message: Finish off rev. 1
Routing:
- net GND: vias 412 -> 410
Changed lines of the file:
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@@
 			)
 		)
+		(property "LCSC" "C32346"
+			(at 0 0 90)
+			(unlocked yes)
+			(layer "F.Fab")
+			(hide yes)
+			(effects
+				(font
+					(size 1 1)
+					(thickness 0.15)
+				)
+			)
+		)
 		(property ki_fp_filters "Crystal*")
 		(sheetname "/")
@@
 	)
 	(via
-		(at 158.25 72.25)
-		(size 0.5)
-		(drill 0.3)
-		(layers "F.Cu" "B.Cu")
-		(free yes)
-		(net 1)
-	)
-	(via
 		(at 150.2 110.1)
 		(size 0.5)
@@
 	)
 	(via
-		(at 157.25 72.25)
-		(size 0.5)
-		(drill 0.3)
-		(layers "F.Cu" "B.Cu")
-		(free yes)
-		(net 1)
-	)
-	(via
 		(at 155 120.5)
 		(size 0.5)
@@
 		(width 0.16)
 		(layer "F.Cu")
-		(net 2)
-	)
-	(segment
-		(start 144.7 102.4)
-		(end 144.6 102.4)
-		(width 0.16)
-		(layer "F.Cu")
